File: EDA files/RCboat.kicad_pcb (KiCad board)
At the start: 2 copper layers, 45.5 x 50 mm, 45 parts, among them J1 Conn_02x10_Odd_Even, J2 Battery, J3 Battery, M1 Motor_Servo, M2 Motor_Servo, SW1 SW_Push, SW2 SW_SPDT, U1 BD9G341EFJ, U2 AMS1117-3.3, U3 NRF24L01_Breakout, U4 STM32F100C4Tx, U5 MPU-6000, Y1 8.000MHZ

Commit message: Add files via upload
Other:
- board text added: "°"
Changed lines of the file:
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@@
   (gr_circle (center 117.7036 105.1) (end 118.237 105.4302) (layer "Edge.Cuts") (width 0.1) (fill none))
   (gr_circle (center 159.9 81.5) (end 160.4334 81.8302) (layer "Edge.Cuts") (width 0.1) (fill none))
+  (gr_text "°" (at 142.8 101.4) (layer "F.SilkS")
+    (effects (font (size 1 1) (thickness 0.25)))
+  )
+  (gr_text "°" (at 142 87.8) (layer "F.SilkS")
+    (effects (font (size 1 1) (thickness 0.25)))
+  )
   (segment (start 124.5 102) (end 127 102) (width 0.2) (layer "F.Cu") (net 1))
   (segment (start 127 102) (end 130.25 98.75) (width 0.2) (layer "F.Cu") (net 1))
